File: hardware/Cyberboard.kicad_sch (KiCad schematic)
At the start: 69 parts, among them J1 Conn_01x20, J2 Conn_01x20, SW1 SW_Push, SW2 SW_Push, U1 SZYY0402Y_C434450, U10 XL-1005UBC_C22355736, U2 TPD2EUSB30, U3 NX2012SA-32.768KHZ-STD-MUB-2, U4 STM32WB55RGVx, U5 BQ24072RGT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

Commit message: it works!!
Connections:
- net GND: no longer U8.6 (CSB)
- no-connect marks 7 -> 8
Changed lines of the file:
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@@
-	)
-	(junction
-		(at 378.46 58.42)
-		(diameter 0)
-		(color 0 0 0 0)
 	)
 	(junction
@@
 	)
 	(no_connect
+		(at 367.03 58.42)
+	)
+	(no_connect
 		(at 255.27 252.73)
 	)
@@
 		)
 		(stroke
-			(width 0)
-			(type default)
-		)
-	)
-	(wire
-		(pts
-			(xy 367.03 58.42) (xy 378.46 58.42)
-		)
-		(stroke
